Commit message: mh2机械臂动作

File: src/mh2_moveit_config/config/robot_urdf.ros2_control.xacro (robot description, xacro)
@@ -8,4 +8,12 @@
                 <plugin>mock_components/GenericSystem</plugin>
             </hardware>
+            <joint name="joint_la0">
+                <command_interface name="position"/>
+                <command_interface name="velocity"/>
+                <state_interface name="position">
+                  <param name="initial_value">${initial_positions['joint_la0']}</param>
+                </state_interface>
+                <state_interface name="velocity"/>
+            </joint>
             <joint name="joint_la1">
                 <command_interface name="position"/>
@@ -61,4 +69,12 @@
                 <state_interface name="position">
                   <param name="initial_value">${initial_positions['joint_la7']}</param>
+                </state_interface>
+                <state_interface name="velocity"/>
+            </joint>
+            <joint name="joint_ra0">
+                <command_interface name="position"/>
+                <command_interface name="velocity"/>
+                <state_interface name="position">
+                  <param name="initial_value">${initial_positions['joint_ra0']}</param>
                 </state_interface>
                 <state_interface name="velocity"/>
